File: PCB/TTT4280_PCB/TTT4280_PCB.kicad_pcb (KiCad board)
At the start: 2 copper layers, 65 x 56 mm, 24 parts, among them J1 Raspberry Pi 3B+ Header, U1 MCP3201-CI/P, U2 MCP3201-CI/P, U3 MCP3201-CI/P, U4 MCP3201-CI/P, U5 MCP3201-CI/P

Commit message: Made updates to PCB, schematic done.
Parts:
- removed L1: DKFP-G22G-D5J0, Vault:DKFPG22GD5J0
- added C14: 1nF, Capacitor_SMD:C_0603_1608Metric_Pad1.08x0.95mm_HandSolder, F.Cu at (148.5, 130.6)
- added C15: 1nF, Capacitor_SMD:C_0603_1608Metric_Pad1.08x0.95mm_HandSolder, F.Cu at (156.3, 124.8)
- added C16: 45.5uF, Capacitor_SMD:C_0603_1608Metric_Pad1.08x0.95mm_HandSolder, F.Cu at (146.5, 130.6)
- added C17: 45.5uF, Capacitor_SMD:C_0603_1608Metric_Pad1.08x0.95mm_HandSolder, F.Cu at (154.3, 124.8)
- added C18: 100nF, Capacitor_SMD:C_0603_1608Metric_Pad1.08x0.95mm_HandSolder, F.Cu at (148.4, 112.7)
- added C19: 100nF, Capacitor_SMD:C_0603_1608Metric_Pad1.08x0.95mm_HandSolder, F.Cu at (97.5, 67.9)
- added C19: 5.7nF, Capacitor_SMD:C_0603_1608Metric_Pad1.08x0.95mm_HandSolder, F.Cu at (137.2, 116.1)
- added C20: 5.7nF, Capacitor_SMD:C_0603_1608Metric_Pad1.08x0.95mm_HandSolder, F.Cu at (153.6, 119.3)
- added C20: 100nF, Capacitor_SMD:C_0603_1608Metric_Pad1.08x0.95mm_HandSolder, F.Cu at (97.5, 70.4)
- added C21: 100nF, Capacitor_SMD:C_0603_1608Metric_Pad1.08x0.95mm_HandSolder, F.Cu at (140.4, 108.6)
- added J2: Conn_01x02_Pin, Connector_PinHeader_2.54mm:PinHeader_1x02_P2.54mm_Vertical, F.Cu at (155.1, 130.8)
- added R1: 1k, Resistor_SMD:R_0603_1608Metric_Pad0.98x0.95mm_HandSolder, F.Cu at (150.5, 130.6)
- added R10: 10k, Resistor_SMD:R_0603_1608Metric_Pad0.98x0.95mm_HandSolder, F.Cu at (101.8, 77.9)
- added R2: 1k, Resistor_SMD:R_0603_1608Metric_Pad0.98x0.95mm_HandSolder, F.Cu at (158.7, 124.8)
- added R3: 1k, Resistor_SMD:R_0603_1608Metric_Pad0.98x0.95mm_HandSolder, F.Cu at (144.5, 130.6)
- added R4: 1k, Resistor_SMD:R_0603_1608Metric_Pad0.98x0.95mm_HandSolder, F.Cu at (152.3, 124.8)
- added R5: 10k, Resistor_SMD:R_0603_1608Metric_Pad0.98x0.95mm_HandSolder, F.Cu at (139.2, 116.1)
- added R6: 10k, Resistor_SMD:R_0603_1608Metric_Pad0.98x0.95mm_HandSolder, F.Cu at (151.8, 119.3)
- added R7: 10k, Resistor_SMD:R_0603_1608Metric_Pad0.98x0.95mm_HandSolder, F.Cu at (101.8, 70.4)
- added R7: 10k, Resistor_SMD:R_0603_1608Metric_Pad0.98x0.95mm_HandSolder, F.Cu at (144.5, 111.6)
- added R8: 10k, Resistor_SMD:R_0603_1608Metric_Pad0.98x0.95mm_HandSolder, F.Cu at (140.4, 111.6)
- added R8: 10k, Resistor_SMD:R_0603_1608Metric_Pad0.98x0.95mm_HandSolder, F.Cu at (101.8, 72.9)
- added R9: 10k, Resistor_SMD:R_0603_1608Metric_Pad0.98x0.95mm_HandSolder, F.Cu at (101.8, 75.4)
- added U10: MCP6002-xMC, Package_DIP:DIP-8_W7.62mm, F.Cu at (141.7, 115.2)
- added U6: MAX4466, Connector_PinHeader_2.54mm:PinHeader_1x03_P2.54mm_Vertical, F.Cu at (102.7, 106.3)
- added U7: MAX4466, Connector_PinHeader_2.54mm:PinHeader_1x03_P2.54mm_Vertical, F.Cu at (93.6, 106.3)
- added U8: MCP3201, Package_DIP:DIP-8_W7.62mm, F.Cu at (151.1, 87.0)
- added U9: MAX4466, Connector_PinHeader_2.54mm:PinHeader_1x03_P2.54mm_Vertical, F.Cu at (98.2, 106.3)
- C1: value ECA1EM101 -> 1uF; footprint Vault:CAPPR55-250-1120X630X1220 -> Capacitor_SMD:C_0603_1608Metric_Pad1.08x0.95mm_HandSolder
- C10, C11, C12, C13, C6, C7, C8, C9: value 7110918 -> 1uF; footprint Vault:CAPPR55-200-1100X500X1200 -> Capacitor_SMD:C_0603_1608Metric_Pad1.08x0.95mm_HandSolder
- C2: value ECA1CM471 -> 1uF; footprint Vault:CAPPR65-350-1150X800X1250 -> Capacitor_SMD:C_0603_1608Metric_Pad1.08x0.95mm_HandSolder
- C3: value C320C104K1R5TA -> 100uF; footprint Vault:C320C104K1R5TA -> Capacitor_SMD:C_0603_1608Metric_Pad1.08x0.95mm_HandSolder
- C4: value 7110918 -> 100uF; footprint Vault:CAPPR55-200-1100X500X1200 -> Capacitor_SMD:C_0603_1608Metric_Pad1.08x0.95mm_HandSolder
- C5: value 7110918 -> 100nF; footprint Vault:CAPPR55-200-1100X500X1200 -> Capacitor_SMD:C_0603_1608Metric_Pad1.08x0.95mm_HandSolder
- J1: value Raspberry Pi 3B+ Header -> Raspberry_Pi_2_3; footprint Vault:HDRV40W85P254_2X20_5080X500X860P -> Connector_PinHeader_2.54mm:PinHeader_2x20_P2.54mm_Vertical
- U1, U2, U3, U4: value MCP3201-CI/P -> MCP3201; footprint Vault:MCHP-P-8 -> Package_DIP:DIP-8_W7.62mm
- U5: value MCP3201-CI/P -> K-LC6; footprint Vault:MCHP-P-8 -> Connector_PinSocket_2.54mm:PinSocket_1x05_P2.54mm_Horizontal; moved to B.Cu
- moved C11 89.7 mm to (93.1, 70.4), turned to 0 degrees
- moved C9 79.0 mm to (88.8, 88.0), turned to 0 degrees
- moved C7 63.3 mm to (88.8, 83.0), turned to 0 degrees
- moved C2 60.6 mm to (88.8, 70.4), turned to 0 degrees
- moved C3 53.2 mm to (88.8, 72.9)
- moved C5 47.9 mm to (88.8, 77.9), turned to 0 degrees
- moved U2 41.3 mm to (165.1, 126.6), turned to 90 degrees
- moved C4 33.0 mm to (88.8, 75.4), turned to 0 degrees
- moved C13 32.8 mm to (161.1, 87.8), turned to -90 degrees
- moved C12 26.3 mm to (148.7, 87.8), turned to -90 degrees
- moved U4 23.9 mm to (165.1, 112.6), turned to 90 degrees
- moved U3 23.2 mm to (137.1, 87.0)
- moved U5 23.0 mm to (173.4, 130.8), turned to 90 degrees
- moved C10 21.8 mm to (147.1, 87.8)
- moved C8 18.5 mm to (134.7, 87.8)
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Connections:
- net DATA1 renamed /DATA1
- C1 pad 1: 3v3_rpi -> +3V3
- C10 pad 1: 3v3 -> +3V3
- C11 pad 1: 3v3 -> +3V3
- C12 pad 1: 3v3 -> +3V3
- C13 pad 1: 3v3 -> +3V3
- C2 pad 1: 3v3 -> +3V3
- C3 pad 1: 3v3 -> +3V3
- C4 pad 1: 3v3 -> +3V3
- C5 pad 1: 3v3 -> GND
- C5 pad 2: GND -> +3V3
- C6 pad 1: 3v3 -> +3V3
- C7 pad 1: 3v3 -> +3V3
- C8 pad 1: 3v3 -> +3V3
- C9 pad 1: 3v3 -> +3V3
- J1 pad 1: 3v3_rpi -> +3V3
- J1 pad 10: (no net) -> unconnected-(J1-GPIO15/RXD-Pad10)
- J1 pad 11: (no net) -> unconnected-(J1-GPIO17-Pad11)
- J1 pad 12: (no net) -> unconnected-(J1-GPIO18/PWM0-Pad12)
- J1 pad 13: DATA5 -> /DATA5
- J1 pad 15: (no net) -> unconnected-(J1-GPIO22-Pad15)
- J1 pad 17: 3v3_rpi -> +3V3
- J1 pad 18: DATA2 -> /DATA2
- J1 pad 19: (no net) -> unconnected-(J1-MOSI0/GPIO10-Pad19)
- J1 pad 2: (no net) -> unconnected-(J1-5V-Pad2)_1
- J1 pad 21: (no net) -> unconnected-(J1-MISO0/GPIO9-Pad21)
- J1 pad 22: DATA3 -> /DATA3
- J1 pad 23: CLK -> /CLK
- J1 pad 24: ~{CS} -> /~{CS}
- J1 pad 26: (no net) -> unconnected-(J1-~{CE1}/GPIO7-Pad26)
- J1 pad 27: (no net) -> unconnected-(J1-ID_SD/GPIO0-Pad27)
- J1 pad 28: (no net) -> unconnected-(J1-ID_SC/GPIO1-Pad28)
- J1 pad 29: (no net) -> unconnected-(J1-GCLK1/GPIO5-Pad29)
- J1 pad 3: (no net) -> unconnected-(J1-SDA/GPIO2-Pad3)
- J1 pad 31: (no net) -> unconnected-(J1-GCLK2/GPIO6-Pad31)
- J1 pad 32: (no net) -> unconnected-(J1-PWM0/GPIO12-Pad32)
- J1 pad 33: (no net) -> unconnected-(J1-PWM1/GPIO13-Pad33)
- J1 pad 35: (no net) -> unconnected-(J1-GPIO19/MISO1-Pad35)
- J1 pad 36: (no net) -> unconnected-(J1-GPIO16-Pad36)
- J1 pad 37: DATA4 -> /DATA4
- J1 pad 38: (no net) -> unconnected-(J1-GPIO20/MOSI1-Pad38)
- J1 pad 4: (no net) -> unconnected-(J1-5V-Pad2)
- J1 pad 40: (no net) -> unconnected-(J1-GPIO21/SCLK1-Pad40)
- J1 pad 5: (no net) -> unconnected-(J1-SCL/GPIO3-Pad5)
- J1 pad 7: (no net) -> unconnected-(J1-GCLK0/GPIO4-Pad7)
- J1 pad 8: (no net) -> unconnected-(J1-GPIO14/TXD-Pad8)
- U1 pad 1: 3v3 -> +3V3
- U1 pad 2: (no net) -> /MIC1
- U1 pad 5: ~{CS} -> /~{CS}
- U1 pad 7: CLK -> /CLK
- U1 pad 8: 3v3 -> +3V3
- U2 pad 1: 3v3 -> +3V3
- U2 pad 2: (no net) -> /filtered_I
- U2 pad 5: ~{CS} -> /~{CS}
- U2 pad 6: DATA2 -> /DATA4
- U2 pad 7: CLK -> /CLK
- U2 pad 8: 3v3 -> +3V3
- U3 pad 1: 3v3 -> +3V3
- U3 pad 2: (no net) -> /MIC2
- U3 pad 5: ~{CS} -> /~{CS}
- U3 pad 6: DATA3 -> /DATA2
- U3 pad 7: CLK -> /CLK
- U3 pad 8: 3v3 -> +3V3
- U4 pad 1: 3v3 -> +3V3
- U4 pad 2: (no net) -> /filtered_Q
- U4 pad 5: ~{CS} -> /~{CS}
- U4 pad 6: DATA4 -> /DATA5
- U4 pad 7: CLK -> /CLK
- U4 pad 8: 3v3 -> +3V3
- U5 pad 1: 3v3 -> /IF_Q
- U5 pad 2: (no net) -> +5V
- U5 pad 3: GND -> /IF_I
- U5 pad 5: ~{CS} -> unconnected-(U5-VCO_in-Pad5)
Routing:
- net GND: track 0.00 -> 93.3 mm
- net /IF_I: track 0.00 -> 23.4 mm
- net +3V3: track 0.00 -> 21.3 mm
- net Net-(U10A--): track 0.00 -> 18.8 mm
- net /IF_Q: track 0.00 -> 17.7 mm
- net +5V: track 0.00 -> 17.1 mm
- net +1V65: track 0.00 -> 16.3 mm
- net Net-(U10B--): track 0.00 -> 11.0 mm
- net /filtered_Q: track 0.00 -> 4.57 mm
- net /filtered_I: track 0.00 -> 4.55 mm
- net Net-(C16-Pad2): track 0.00 -> 2.74 mm
